File: AX5043/SDRMod.sch (KiCad schematic (older format))
At the start: 44 parts, among them P1 CONN_02X06, Q1 Q_NPN_BCE, Q2 RE1C002UNTCL, Q3 RE1C002UNTCL, Q4 RE1C002UNTCL, Q5 RE1C002UNTCL, Q6 RE1C002UNTCL, U1 AX5043, Y1 Crystal

Commit message: AX5043 and level shifter splitted into two projects, IR removed
Parts:
- removed C7, C8: C, Capacitors_SMD:C_0603_HandSoldering, symbol C
- removed D1: LED, LEDs:LED_D3.0mm, symbol LED
- removed NA1: L, Inductors_SMD:L_0603_HandSoldering, symbol L
- removed P1: CONN_02X06, Pin_Headers:Pin_Header_Straight_2x06_Pitch2.00mm, symbol CONN_02X06
- removed Q1: Q_NPN_BCE, TO_SOT_Packages_SMD:SOT-23_Handsoldering, symbol Q_NPN_BCE
- removed Q2, Q3, Q4, Q5, Q6: RE1C002UNTCL, TO_SOT_Packages_SMD:SOT-23_Handsoldering, symbol Q_NMOS_DGS
- removed R1, R2: R, Resistors_SMD:R_0603_HandSoldering, symbol R
- removed RN1, RN2: R_Network05, TO_SOT_Packages_SMD:SOT-23-6_Handsoldering, symbol R_Network05
- added P1: CONN_02X04, Pin_Headers:Pin_Header_Straight_2x04_Pitch2.00mm_SMD, symbol CONN_02X04
Connections:
- net labels removed: +1V8, DATA, DCLK, IR1, MuC_Interrupt_IN, MuC_SPI1_CS0, MuC_SPI1_MISO, MuC_SPI1_MOSI, MuC_SPI1_SCK, SYSCLK
- wire segments 142 -> 91
- no-connect marks 7 -> 11
Other:
- moved on the sheet: C10, C11, C9
